File: src/solder-ships.kicad_sch (KiCad schematic)
At the start: 5 parts, among them Q1 KPS-3227, Q2 NPN

Commit message: start wiring
Parts:
- removed Q2: NPN, symbol Simulation_SPICE:NPN
- added Q2: PNP, symbol Simulation_SPICE:PNP
Connections:
- net at Q1.1, Q1.3: now also BT1.2 (-), Q2.3 (E)
- net at Q1.2, Q1.4: now also Q2.2 (B)
Other:
- moved on the sheet: C1, D1, Q1
Changed lines of the file:
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@@
 	(generator_version "9.0")
 	(paper "A4")
+	(junction
+		(at 123.19 127)
+		(diameter 0)
+		(color 0 0 0 0)
+	)
+	(wire
+		(pts
+			(xy 123.19 127) (xy 123.19 140.97)
+		)
+		(stroke
+			(width 0)
+			(type default)
+		)
+	)
+	(wire
+		(pts
+			(xy 168.91 140.97) (xy 168.91 132.08)
+		)
+		(stroke
+			(width 0)
+			(type default)
+		)
+	)
+	(wire
+		(pts
+			(xy 123.19 127) (xy 138.43 127)
+		)
+		(stroke
+			(width 0)
+			(type default)
+		)
+	)
+	(wire
+		(pts
+			(xy 123.19 140.97) (xy 168.91 140.97)
+		)
+		(stroke
+			(width 0)
+			(type default)
+		)
+	)
+	(wire
+		(pts
+			(xy 148.59 127) (xy 161.29 127)
+		)
+		(stroke
+			(width 0)
+			(type default)
+		)
+	)
+	(wire
+		(pts
+			(xy 123.19 118.11) (xy 123.19 127)
+		)
+		(stroke
+			(width 0)
+			(type default)
+		)
+	)
 	(symbol
 		(lib_id "Sensor_Optical:KPS-3227")
-		(at 162.56 91.44 0)
+		(at 143.51 127 90)
 		(unit 1)
 		(exclude_from_sim no)
@@
 		(fields_autoplaced yes)
 		(property "Reference" "Q1"
-			(at 165.1 89.4206 0)
-			(effects
-				(font
-					(size 1.27 1.27)
-				)
-				(justify left)
+			(at 142.7607 120.65 90)
+			(effects
+				(font
+					(size 1.27 1.27)
+				)
 			)
 		)
 		(property "Value" "KPS-3227"
-			(at 165.1 91.9606 0)
-			(effects
-				(font
-					(size 1.27 1.27)
-				)
-				(justify left)
+			(at 142.7607 123.19 90)
+			(effects
+				(font
+					(size 1.27 1.27)
+				)
 			)
 		)
 		(property "Footprint" "OptoDevice:Kingbright_KPS-3227"
-			(at 162.56 87.63 0)
+			(at 139.7 127 0)
 			(effects
 				(font
@@
 		)
 		(property "Datasheet" "https://www.kingbright.com/attachments/file/psearch/000/00/00/KPS-3227SP1C(Ver.16).pdf"
-			(at 162.56 87.63 0)
+			(at 139.7 127 0)
 			(effects
 				(font
@@
 		)
 		(property "Description" "Ambient light NPN phototransistor, KPS-3227"
-			(at 162.56 91.44 0)
+			(at 143.51 127 0)
 			(effects
 				(font
@@
 	)
 	(symbol
+		(lib_id "Simulation_SPICE:PNP")
+		(at 166.37 127 0)
+		(unit 1)
+		(exclude_from_sim no)
+		(in_bom yes)
+		(on_board yes)
+		(dnp no)
+		(fields_autoplaced yes)
+		(property "Reference" "Q2"
+			(at 171.45 125.7299 0)
+			(effects
+				(font
+					(size 1.27 1.27)
+				)
+				(justify left)
+			)
+		)
+		(property "Value" "PNP"
+			(at 171.45 128.2699 0)
+			(effects
+				(font
+					(size 1.27 1.27)
+				)
+				(justify left)
+			)
+		)
+		(property "Footprint" ""
+			(at 201.93 127 0)
+			(effects
+				(font
+					(size 1.27 1.27)
+				)
+				(hide yes)
+			)
+		)
+		(property "Datasheet" "https://ngspice.sourceforge.io/docs/ngspice-html-manual/manual.xhtml#cha_BJTs"
+			(at 201.93 127 0)
+			(effects
+				(font
+					(size 1.27 1.27)
+				)
+				(hide yes)
+			)
+		)
+		(property "Description" "Bipolar transistor symbol for simulation only, substrate tied to the emitter"
+			(at 166.37 127 0)
+			(effects
+				(font
+					(size 1.27 1.27)
+				)
+				(hide yes)
+			)
+		)
+		(property "Sim.Device" "PNP"
+			(at 166.37 127 0)
+			(effects
+				(font
+					(size 1.27 1.27)
+				)
+				(hide yes)
+			)
+		)
+		(property "Sim.Type" "GUMMELPOON"
+			(at 166.37 127 0)
+			(effects
+				(font
+					(size 1.27 1.27)
+				)
+				(hide yes)
+			)
+		)
+		(property "Sim.Pins" "1=C 2=B 3=E"
+			(at 166.37 127 0)
+			(effects
+				(font
+					(size 1.27 1.27)
+				)
+				(hide yes)
+			)
+		)
+		(pin "1"
+		)
+		(pin "2"
+		)
+		(pin "3"
+		)
+		(instances
+			(project ""
+				(path "/67ea8089-b1c4-4ff2-8f17-3c25f880c6b4"
+					(reference "Q2")
+					(unit 1)
+				)
+			)
+		)
+	)
+	(symbol
 		(lib_id "Device:LED")
-		(at 167.64 115.57 0)
+		(at 160.02 102.87 0)
 		(unit 1)
 		(exclude_from_sim no)
@@
 		(fields_autoplaced yes)
 		(property "Reference" "D1"
-			(at 166.0525 109.22 0)
+			(at 158.4325 96.52 0)
 			(effects
 				(font
@@
 		)
 		(property "Value" "LED"
-			(at 166.0525 111.76 0)
+			(at 158.4325 99.06 0)
 			(effects
 				(font
@@
 		)
 		(property "Footprint" ""
-			(at 167.64 115.57 0)
+			(at 160.02 102.87 0)
 			(effects
 				(font
@@
 		)
 		(property "Datasheet" "~"
-			(at 167.64 115.57 0)
+			(at 160.02 102.87 0)
 			(effects
 				(font
@@
 		)
 		(property "Description" "Light emitting diode"
-			(at 167.64 115.57 0)
+			(at 160.02 102.87 0)
 			(effects
 				(font
@@
 		)
 		(property "Sim.Pins" "1=K 2=A"
-			(at 167.64 115.57 0)
+			(at 160.02 102.87 0)
 			(effects
 				(font
@@
 	)
 	(symbol
-		(lib_id "Simulation_SPICE:NPN")
-		(at 161.29 130.81 0)
-		(unit 1)
-		(exclude_from_sim no)
-		(in_bom yes)
-		(on_board yes)
-		(dnp no)
-		(fields_autoplaced yes)
-		(property "Reference" "Q2"
-			(at 166.37 129.5399 0)
-			(effects
-				(font
-					(size 1.27 1.27)
-				)
-				(justify left)
-			)
-		)
-		(property "Value" "NPN"
-			(at 166.37 132.0799 0)
-			(effects
-				(font
-					(size 1.27 1.27)
-				)
-				(justify left)
-			)
-		)
-		(property "Footprint" ""
-			(at 224.79 130.81 0)
-			(effects
-				(font
-					(size 1.27 1.27)
-				)
-				(hide yes)
-			)
-		)
-		(property "Datasheet" "https://ngspice.sourceforge.io/docs/ngspice-html-manual/manual.xhtml#cha_BJTs"
-			(at 224.79 130.81 0)
-			(effects
-				(font
-					(size 1.27 1.27)
-				)
-				(hide yes)
-			)
-		)
-		(property "Description" "Bipolar transistor symbol for simulation only, substrate tied to the emitter"
-			(at 161.29 130.81 0)
-			(effects
-				(font
-					(size 1.27 1.27)
-				)
-				(hide yes)
-			)
-		)
-		(property "Sim.Device" "NPN"
-			(at 161.29 130.81 0)
-			(effects
-				(font
-					(size 1.27 1.27)
-				)
-				(hide yes)
-			)
-		)
-		(property "Sim.Type" "GUMMELPOON"
-			(at 161.29 130.81 0)
-			(effects
-				(font
-					(size 1.27 1.27)
-				)
-				(hide yes)
-			)
-		)
-		(property "Sim.Pins" "1=C 2=B 3=E"
-			(at 161.29 130.81 0)
-			(effects
-				(font
-					(size 1.27 1.27)
-				)
-				(hide yes)
-			)
-		)
-		(pin "1"
-		)
-		(pin "3"
-		)
-		(pin "2"
-		)
-		(instances
-			(project ""
-				(path "/67ea8089-b1c4-4ff2-8f17-3c25f880c6b4"
-					(reference "Q2")
-					(unit 1)
-				)
-			)
-		)
-	)
-	(symbol
 		(lib_id "Device:C_Small_US")
-		(at 125.73 135.89 0)
+		(at 149.86 111.76 0)
 		(unit 1)
 		(exclude_from_sim no)
@@
 		(fields_autoplaced yes)
 		(property "Reference" "C1"
-			(at 128.27 134.7469 0)
+			(at 152.4 110.6169 0)
 			(effects
 				(font
@@
 		)
 		(property "Value" "C_Small_US"
-			(at 128.27 137.2869 0)
+			(at 152.4 113.1569 0)
 			(effects
 				(font
@@
 		)
 		(property "Footprint" ""
-			(at 125.73 135.89 0)
+			(at 149.86 111.76 0)
 			(effects
 				(font
@@
 		)
 		(property "Datasheet" ""
-			(at 125.73 135.89 0)
+			(at 149.86 111.76 0)
 			(effects
 				(font
@@
 		)
 		(property "Description" "capacitor, small US symbol"
-			(at 125.73 135.89 0)
-			(effects
-				(font
+			(at 149.86 111.76 0)
+			(effects
+				(font

Commit message: IDK what I should make
Parts:
- removed C1: C_Small_US, symbol Device:C_Small_US
- removed D1: LED, symbol Device:LED
- removed Q1: KPS-3227, OptoDevice:Kingbright_KPS-3227, symbol Sensor_Optical:KPS-3227
- removed Q2: PNP, symbol Simulation_SPICE:PNP
- added Q1: Q_NPN, symbol Device:Q_NPN
- added Q2, Q3, Q4: NPN, symbol Simulation_SPICE:NPN
- added R1: R, symbol Device:R
Other:
- moved on the sheet: BT1

Commit message: Let's save footprints for tomorrow...
Parts:
- removed Q1: Q_NPN, symbol Device:Q_NPN
- added D1, D2, D3, D4, D5, D6: LED, symbol Device:LED
- added Q1, Q5, Q6: NPN, symbol Simulation_SPICE:NPN
- added R10, R11, R12, R13, R14, R15, R4, R5, R6, R7: 4.7k, symbol Device:R
- added R16, R8, R9: 47k, symbol Device:R
- added R2: R_Photo, symbol Device:R_Photo
- added R3: 220, symbol Device:R
- BT1: footprint (none) -> Battery:BatteryHolder_Multicomp_BC-2001_1x2032
- R1: value R -> 47k
Connections:
- net at Q4.1 (C): now also D4.1 (K)
- net at Q4.2 (B): now also R13.1
- net at Q4.3 (E): now also BT1.2 (-), Q2.3 (E), Q3.3 (E), Q1.3 (E), Q5.3 (E), Q6.3 (E), R2.2
- net at Q2.1 (C): now also D3.1 (K)
- net at Q2.2 (B): now also R5.1
- net at Q3.1 (C): now also D2.1 (K)
- net at Q3.2 (B): now also R11.1
- net at R1.1: now also R10.2, R2.1, R4.2, R6.2, R7.2, R8.2, R9.2
- net at R1.2: now also BT1.1 (+), R3.2
- new net: D1.2 (A), D2.2 (A), D3.2 (A), D4.2 (A), D5.2 (A), D6.2 (A), R3.1
- new net: D1.1 (K), Q1.1 (C)
- new net: D5.1 (K), Q6.1 (C)
- new net: Q6.2 (B), R16.1
- new net: R13.2, R14.1
- new net: R14.2, R15.1
- new net: D6.1 (K), Q5.1 (C)
- new net: R12.2, R6.1
- new net: R15.2, R7.1
- new net: R11.2, R12.1
- new net: Q5.2 (B), R8.1
- new net: R16.2, R9.1
- new net: R10.1, R5.2
- new net: Q1.2 (B), R4.1
Other:
- title: (none) -> Sequential Lights
- moved on the sheet: BT1, R1

Commit message: Add footprints
Parts:
- D1, D2, D3, D4, D5, D6: footprint (none) -> LED_THT:LED_D5.0mm
- Q1, Q2, Q3, Q4, Q5, Q6: footprint (none) -> Package_TO_SOT_THT:TO-92L_HandSolder
- R1, R10, R11, R12, R13, R14, R15, R16, R3, R4, R5, R6, R7, R8, R9: footprint (none) -> Resistor_THT:R_Axial_DIN0207_L6.3mm_D2.5mm_P7.62mm_Horizontal
- R2: footprint (none) -> Potentiometer_THT:Potentiometer_Vishay_T73YP_Vertical
Changed lines of the file:
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@@
 			)
 		)
-		(property "Footprint" ""
+		(property "Footprint" "LED_THT:LED_D5.0mm"
 			(at 118.11 102.87 0)
 			(effects
@@
 			)
 		)
-		(property "Footprint" ""
+		(property "Footprint" "LED_THT:LED_D5.0mm"
 			(at 118.11 35.56 0)
 			(effects
@@
 			)
 		)
-		(property "Footprint" ""
+		(property "Footprint" "Package_TO_SOT_THT:TO-92L_HandSolder"
 			(at 140.97 85.09 0)
 			(effects
@@
 			)
 		)
-		(property "Footprint" ""
+		(property "Footprint" "Resistor_THT:R_Axial_DIN0207_L6.3mm_D2.5mm_P7.62mm_Horizontal"
 			(at 173.99 112.268 90)
 			(effects
@@
 			)
 		)
-		(property "Footprint" ""
+		(property "Footprint" "LED_THT:LED_D5.0mm"
 			(at 118.11 125.73 0)
 			(effects
@@
 			)
 		)
-		(property "Footprint" ""
+		(property "Footprint" "Resistor_THT:R_Axial_DIN0207_L6.3mm_D2.5mm_P7.62mm_Horizontal"
 			(at 200.66 90.678 90)
 			(effects
@@
 			)
 		)
-		(property "Footprint" ""
+		(property "Footprint" "Potentiometer_THT:Potentiometer_Vishay_T73YP_Vertical"
 			(at 66.04 45.72 90)
 			(effects
@@
 			)
 		)
-		(property "Footprint" ""
+		(property "Footprint" "Resistor_THT:R_Axial_DIN0207_L6.3mm_D2.5mm_P7.62mm_Horizontal"
 			(at 187.96 112.268 90)
 			(effects
@@
 			)
 		)
-		(property "Footprint" ""
+		(property "Footprint" "Resistor_THT:R_Axial_DIN0207_L6.3mm_D2.5mm_P7.62mm_Horizontal"
 			(at 158.75 112.268 90)
 			(effects
@@
 			)
 		)
-		(property "Footprint" ""
+		(property "Footprint" "Resistor_THT:R_Axial_DIN0207_L6.3mm_D2.5mm_P7.62mm_Horizontal"
 			(at 160.02 90.678 90)
 			(effects
@@
 			)
 		)
-		(property "Footprint" ""
+		(property "Footprint" "Package_TO_SOT_THT:TO-92L_HandSolder"
 			(at 140.97 64.77 0)
 			(effects
@@
 			)
 		)
-		(property "Footprint" ""
+		(property "Footprint" "LED_THT:LED_D5.0mm"
 			(at 118.11 146.05 0)
 			(effects
@@
 			)
 		)
-		(property "Footprint" ""
+		(property "Footprint" "Package_TO_SOT_THT:TO-92L_HandSolder"
 			(at 140.97 41.91 0)
 			(effects
@@
 			)
 		)
-		(property "Footprint" ""
+		(property "Footprint" "Package_TO_SOT_THT:TO-92L_HandSolder"
 			(at 140.97 20.32 0)
 			(effects
@@
 			)
 		)
-		(property "Footprint" ""
+		(property "Footprint" "Resistor_THT:R_Axial_DIN0207_L6.3mm_D2.5mm_P7.62mm_Horizontal"
 			(at 167.64 155.448 90)
 			(effects
@@
 			)
 		)
-		(property "Footprint" ""
+		(property "Footprint" "Resistor_THT:R_Axial_DIN0207_L6.3mm_D2.5mm_P7.62mm_Horizontal"
 			(at 180.34 90.678 90)
 			(effects
@@
 			)
 		)
-		(property "Footprint" ""
+		(property "Footprint" "Resistor_THT:R_Axial_DIN0207_L6.3mm_D2.5mm_P7.62mm_Horizontal"
 			(at 162.56 66.548 90)
 			(effects
@@
 			)
 		)
-		(property "Footprint" ""
+		(property "Footprint" "Resistor_THT:R_Axial_DIN0207_L6.3mm_D2.5mm_P7.62mm_Horizontal"
 			(at 88.392 73.66 90)
 			(effects
@@
 			)
 		)
-		(property "Footprint" ""
+		(property "Footprint" "Resistor_THT:R_Axial_DIN0207_L6.3mm_D2.5mm_P7.62mm_Horizontal"
 			(at 190.5 155.448 90)
 			(effects
@@
 			)
 		)
-		(property "Footprint" ""
+		(property "Footprint" "Package_TO_SOT_THT:TO-92L_HandSolder"
 			(at 140.97 -25.4 0)
 			(effects
@@
 			)
 		)
-		(property "Footprint" ""
+		(property "Footprint" "Resistor_THT:R_Axial_DIN0207_L6.3mm_D2.5mm_P7.62mm_Horizontal"
 			(at 179.07 135.128 90)
 			(effects
@@
 			)
 		)
-		(property "Footprint" ""
+		(property "Footprint" "Resistor_THT:R_Axial_DIN0207_L6.3mm_D2.5mm_P7.62mm_Horizontal"
 			(at 176.53 44.958 90)
 			(effects
@@
 			)
 		)
-		(property "Footprint" ""
+		(property "Footprint" "Package_TO_SOT_THT:TO-92L_HandSolder"
 			(at 140.97 -3.81 0)
 			(effects
@@
 			)
 		)
-		(property "Footprint" ""
+		(property "Footprint" "LED_THT:LED_D5.0mm"
 			(at 118.11 81.28 0)
 			(effects
@@
 			)
 		)
-		(property "Footprint" ""
+		(property "Footprint" "LED_THT:LED_D5.0mm"
 			(at 118.11 57.15 0)
 			(effects
@@
 			)
 		)
-		(property "Footprint" ""
+		(property "Footprint" "Resistor_THT:R_Axial_DIN0207_L6.3mm_D2.5mm_P7.62mm_Horizontal"
 			(at 200.66 112.268 90)
 			(effects
@@
 			)
 		)
-		(property "Footprint" ""
+		(property "Footprint" "Resistor_THT:R_Axial_DIN0207_L6.3mm_D2.5mm_P7.62mm_Horizontal"
 			(at 195.58 66.548 90)
 			(effects
@@
 			)
 		)
-		(property "Footprint" ""
+		(property "Footprint" "Resistor_THT:R_Axial_DIN0207_L6.3mm_D2.5mm_P7.62mm_Horizontal"
 			(at 65.532 73.66 90)
 			(effects

Commit message: New Idea
Parts:
- removed D2, D3, D4, D5, D6: LED, LED_THT:LED_D5.0mm, symbol Device:LED
- removed Q2, Q3, Q4, Q5, Q6: NPN, Package_TO_SOT_THT:TO-92L_HandSolder, symbol Simulation_SPICE:NPN
- removed R10, R11, R12, R13, R14, R15, R4, R5, R6, R7: 4.7k, Resistor_THT:R_Axial_DIN0207_L6.3mm_D2.5mm_P7.62mm_Horizontal, symbol Device:R
- removed R16, R8, R9: 47k, Resistor_THT:R_Axial_DIN0207_L6.3mm_D2.5mm_P7.62mm_Horizontal, symbol Device:R
- BT1: footprint Battery:BatteryHolder_Multicomp_BC-2001_1x2032 -> Battery:BatteryHolder_Keystone_3034_1x20mm
- D1: footprint LED_THT:LED_D5.0mm -> (none)
- Q1: footprint Package_TO_SOT_THT:TO-92L_HandSolder -> (none)
- R1: value 47k -> 4.7kΩ
- R2: footprint Potentiometer_THT:Potentiometer_Vishay_T73YP_Vertical -> Resistor_THT:R_Axial_DIN0207_L6.3mm_D2.5mm_P7.62mm_Horizontal
- R3: value 220 -> 220Ω
Connections:
- net at R3.1: now also BT1.1 (+), R1.2; no longer D1.2 (A)
- net at R1.1, R2.1: now also Q1.2 (B)
- new net: D1.2 (A), R3.2
Other:
- title: Sequential Lights -> Sequential Lighting
- moved on the sheet: BT1, R1, R2

Commit message: PCB Design
Parts:
- D1: footprint (none) -> LED_THT:LED_D5.0mm
- Q1: footprint (none) -> Package_TO_SOT_THT:TO-92L_HandSolder
Changed lines of the file:
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@@
 			)
 		)
-		(property "Footprint" ""
+		(property "Footprint" "Package_TO_SOT_THT:TO-92L_HandSolder"
 			(at 243.84 87.63 0)
 			(effects
@@
 			)
 		)
-		(property "Footprint" ""
+		(property "Footprint" "LED_THT:LED_D5.0mm"
 			(at 172.72 107.95 0)
 			(effects
