File: src/solder-ships.kicad_pcb (KiCad board)
At the start: 2 copper layers, 29 parts, among them Q1 NPN, Q2 NPN, Q3 NPN, Q4 NPN, Q5 NPN, Q6 NPN

Commit message: PCB Design
Parts:
- removed D2, D3, D4, D5, D6: LED, LED_THT:LED_D5.0mm
- removed Q2, Q3, Q4, Q5, Q6: NPN, Package_TO_SOT_THT:TO-92L_HandSolder
- removed R10, R11, R12, R13, R14, R15, R4, R5, R6, R7: 4.7k, Resistor_THT:R_Axial_DIN0207_L6.3mm_D2.5mm_P7.62mm_Horizontal
- removed R16, R8, R9: 47k, Resistor_THT:R_Axial_DIN0207_L6.3mm_D2.5mm_P7.62mm_Horizontal
- R1: value 47k -> 4.7kΩ
- R2: footprint Potentiometer_THT:Potentiometer_Vishay_T73YP_Vertical -> Resistor_THT:R_Axial_DIN0207_L6.3mm_D2.5mm_P7.62mm_Horizontal
- R3: value 220 -> 220Ω
- moved R1 65.5 mm to (148.2, 115.4), turned to 90 degrees
- moved D1 64.5 mm to (150.5, 121.8)
- moved R3 52.6 mm to (142.2, 107.9), turned to -90 degrees
- moved Q1 48.2 mm to (162.5, 112.1), turned to 90 degrees
- moved R2 24.7 mm to (154.2, 115.4), turned to 90 degrees
- moved BT1 10.4 mm to (152.1, 94.4)
Connections:
- R1 pad 1: Net-(R1-Pad1) -> Net-(Q1-B)
- R2 pad 1: Net-(R1-Pad1) -> Net-(Q1-B)
- R3 pad 1: Net-(D1-A) -> Net-(BT1-+)
- R3 pad 2: Net-(BT1-+) -> Net-(D1-A)

Commit message: Finish PCB design
Other:
- board outline added: 35 x 63 mm
Changed lines of the file:
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@@
 	)
 	(paper "A4")
+	(title_block
+		(title "Sequential Lighting")
+		(date "2025-04-27")
+		(rev "1.1.1")
+	)
 	(layers
 		(0 "F.Cu" signal)
@@
 		)
 	)
+	(gr_poly
+		(pts
+			(xy 151.75 135) (xy 168.75 119.25) (xy 169.25 86.75) (xy 151.5 72) (xy 134.25 87.75) (xy 134.5 119.25)
+		)
+		(stroke
+			(width 0.05)
+			(type solid)
+		)
+		(fill no)
+		(layer "Edge.Cuts")
+	)
 	(embedded_fonts no)

Commit message: Wire the Board
Parts:
- moved D1 1.79 mm to (152.2, 121.5), turned to 180 degrees
Routing:
- net Net-(BT1-+): track 0.00 -> 66.9 mm
- net Net-(BT1--): track 0.00 -> 23.3 mm
- net Net-(Q1-B): track 0.00 -> 14.9 mm
- net Net-(D1-K): track 0.00 -> 14.1 mm
- net Net-(D1-A): track 0.00 -> 9.92 mm
Changed lines of the file:
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@@
 	(footprint "LED_THT:LED_D5.0mm"
 		(layer "F.Cu")
-		(at 150.475 121.75)
+		(at 152.25 121.5 180)
 		(descr "LED, diameter 5.0mm, 2 pins, http://cdn-reichelt.de/documents/datenblatt/A500/LL-504BC2E-009.pdf, generated by kicad-footprint-generator")
 		(tags "LED")
@@
 		)
 		(property "Sim.Pins" "1=K 2=A"
-			(at 0 0 0)
+			(at 0 0 180)
 			(unlocked yes)
 			(layer "F.Fab")
@@
 		)
 		(fp_arc
+			(start 4.26 0.000048)
+			(mid 2.071756 2.880501)
+			(end -1.29 1.54483)
+			(stroke
+				(width 0.12)
+				(type solid)
+			)
+			(layer "F.SilkS")
+		)
+		(fp_arc
 			(start -1.29 -1.54483)
 			(mid 2.071756 -2.880501)
@@
 			(layer "F.SilkS")
 		)
-		(fp_arc
-			(start 4.26 0.000048)
-			(mid 2.071756 2.880501)
-			(end -1.29 1.54483)
-			(stroke
-				(width 0.12)
-				(type solid)
-			)
-			(layer "F.SilkS")
-		)
 		(fp_circle
 			(center 1.27 0)
@@
 		)
 		(fp_line
+			(start 4.49 3.21)
+			(end 4.49 -3.21)
+			(stroke
+				(width 0.05)
+				(type solid)
+			)
+			(layer "F.CrtYd")
+		)
+		(fp_line
+			(start 4.49 -3.21)
+			(end -1.94 -3.21)
+			(stroke
+				(width 0.05)
+				(type solid)
+			)
+			(layer "F.CrtYd")
+		)
+		(fp_line
+			(start -1.94 3.21)
+			(end 4.49 3.21)
+			(stroke
+				(width 0.05)
+				(type solid)
+			)
+			(layer "F.CrtYd")
+		)
+		(fp_line
 			(start -1.94 -3.21)
 			(end -1.94 3.21)
-			(stroke
-				(width 0.05)
-				(type solid)
-			)
-			(layer "F.CrtYd")
-		)
-		(fp_line
-			(start -1.94 3.21)
-			(end 4.49 3.21)
-			(stroke
-				(width 0.05)
-				(type solid)
-			)
-			(layer "F.CrtYd")
-		)
-		(fp_line
-			(start 4.49 -3.21)
-			(end -1.94 -3.21)
-			(stroke
-				(width 0.05)
-				(type solid)
-			)
-			(layer "F.CrtYd")
-		)
-		(fp_line
-			(start 4.49 3.21)
-			(end 4.49 -3.21)
 			(stroke
 				(width 0.05)
@@
 		)
 		(pad "1" thru_hole rect
-			(at 0 0)
+			(at 0 0 180)
 			(size 1.8 1.8)
 			(drill 0.9)
@@
 		)
 		(pad "2" thru_hole circle
-			(at 2.54 0)
+			(at 2.54 0 180)
 			(size 1.8 1.8)
 			(drill 0.9)
@@
 		(layer "Edge.Cuts")
 	)
+	(segment
+		(start 154.25 96.538075)
+		(end 152.12 94.408075)
+		(width 0.2)
+		(layer "F.Cu")
+		(net 1)
+	)
+	(segment
+		(start 154.25 107.82)
+		(end 154.25 96.538075)
+		(width 0.2)
+		(layer "F.Cu")
+		(net 1)
+	)
+	(segment
+		(start 162.5 109.59)
+		(end 160.73 107.82)
+		(width 0.2)
+		(layer "F.Cu")
+		(net 1)
+	)
+	(segment
+		(start 160.73 107.82)
+		(end 154.25 107.82)
+		(width 0.2)
+		(layer "F.Cu")
+		(net 1)
+	)
+	(segment
+		(start 155.931179 85.207075)
+		(end 163.105 92.380896)
+		(width 0.2)
+		(layer "F.Cu")
+		(net 2)
+	)
+	(segment
+		(start 163.105 92.380896)
+		(end 163.105 94.408075)
+		(width 0.2)
+		(layer "F.Cu")
+		(net 2)
+	)
+	(segment
+		(start 142.919 102.489)
+		(end 142.919 90.596896)
+		(width 0.2)
+		(layer "F.Cu")
+		(net 2)
+	)
+	(segment
+		(start 148.13 107.94)
+		(end 148.25 107.82)
+		(width 0.2)
+		(layer "F.Cu")
+		(net 2)
+	)
+	(segment
+		(start 142.919 90.596896)
+		(end 148.308821 85.207075)
+		(width 0.2)
+		(layer "F.Cu")
+		(net 2)
+	)
+	(segment
+		(start 141.135 94.408075)
+		(end 141.135 106.825)
+		(width 0.2)
+		(layer "F.Cu")
+		(net 2)
+	)
+	(segment
+		(start 148.308821 85.207075)
+		(end 155.931179 85.207075)
+		(width 0.2)
+		(layer "F.Cu")
+		(net 2)
+	)
+	(segment
+		(start 142.25 107.94)
+		(end 148.13 107.94)
+		(width 0.2)
+		(layer "F.Cu")
+		(net 2)
+	)
+	(segment
+		(start 148.25 107.82)
+		(end 142.919 102.489)
+		(width 0.2)
+		(layer "F.Cu")
+		(net 2)
+	)
+	(segment
+		(start 141.135 106.825)
+		(end 142.25 107.94)
+		(width 0.2)
+		(layer "F.Cu")
+		(net 2)
+	)
+	(segment
+		(start 152.25 121.5)
+		(end 153.13 121.5)
+		(width 0.2)
+		(layer "F.Cu")
+		(net 3)
+	)
+	(segment
+		(start 153.13 121.5)
+		(end 162.5 112.13)
+		(width 0.2)
+		(layer "F.Cu")
+		(net 3)
+	)
+	(segment
+		(start 143.77 115.56)
+		(end 149.71 121.5)
+		(width 0.2)
+		(layer "F.Cu")
+		(net 4)
+	)
+	(segment
+		(start 142.25 115.56)
+		(end 143.77 115.56)
+		(width 0.2)
+		(layer "F.Cu")
+		(net 4)
+	)
+	(segment
+		(start 148.25 115.44)
+		(end 154.25 115.44)
+		(width 0.2)
+		(layer "F.Cu")
+		(net 5)
+	)
+	(segment
+		(start 154.25 115.44)
+		(end 156.65 115.44)
+		(width 0.2)
+		(layer "F.Cu")
+		(net 5)
+	)
+	(segment
+		(start 156.65 115.44)
+		(end 161.23 110.86)
+		(width 0.2)
+		(layer "F.Cu")
+		(net 5)
+	)
 	(embedded_fonts no)
